Commit message: g1仿真模型导入

File: unitree_g1_ros2_function_pkg/src/g1_sim/urdf/g1_29dof_with_hand.urdf (robot description, URDF)
Before this commit: robot g1_29dof_with_hand, 54 links, 53 joints
Links:
- link head_link: geometry collision mesh filename=package://g1_sim/meshes/head_link.STL; visual mesh filename=package://g1_sim/meshes/head_link.STL
- link left_ankle_pitch_link: geometry collision mesh filename=package://g1_sim/meshes/left_ankle_pitch_link.STL; visual mesh filename=package://g1_sim/meshes/left_ankle_pitch_link.STL
- link left_ankle_roll_link: geometry collision sphere radius=0.005; collision sphere radius=0.005
- link left_elbow_link: geometry collision mesh filename=package://g1_sim/meshes/left_elbow_link.STL; visual mesh filename=package://g1_sim/meshes/left_elbow_link.STL
- link left_hand_index_0_link: geometry collision mesh filename=package://g1_sim/meshes/left_hand_index_0_link.STL; visual mesh filename=package://g1_sim/meshes/left_hand_index_0_link.STL
- link left_hand_index_1_link: geometry collision mesh filename=package://g1_sim/meshes/left_hand_index_1_link.STL; visual mesh filename=package://g1_sim/meshes/left_hand_index_1_link.STL
- link left_hand_middle_0_link: geometry collision mesh filename=package://g1_sim/meshes/left_hand_middle_0_link.STL; visual mesh filename=package://g1_sim/meshes/left_hand_middle_0_link.STL
- link left_hand_middle_1_link: geometry collision mesh filename=package://g1_sim/meshes/left_hand_middle_1_link.STL; visual mesh filename=package://g1_sim/meshes/left_hand_middle_1_link.STL
- link left_hand_palm_link: geometry collision mesh filename=package://g1_sim/meshes/left_hand_palm_link.STL; visual mesh filename=package://g1_sim/meshes/left_hand_palm_link.STL
- link left_hand_thumb_0_link: geometry collision mesh filename=package://g1_sim/meshes/left_hand_thumb_0_link.STL; visual mesh filename=package://g1_sim/meshes/left_hand_thumb_0_link.STL
- link left_hand_thumb_1_link: geometry collision box size=0.02 0.03 0.02; visual mesh filename=package://g1_sim/meshes/left_hand_thumb_1_link.STL
- link left_hand_thumb_2_link: geometry collision mesh filename=package://g1_sim/meshes/left_hand_thumb_2_link.STL; visual mesh filename=package://g1_sim/meshes/left_hand_thumb_2_link.STL
- link left_hip_pitch_link: geometry collision mesh filename=package://g1_sim/meshes/left_hip_pitch_link.STL; visual mesh filename=package://g1_sim/meshes/left_hip_pitch_link.STL
- link left_hip_roll_link: geometry collision mesh filename=package://g1_sim/meshes/left_hip_roll_link.STL; visual mesh filename=package://g1_sim/meshes/left_hip_roll_link.STL
- link left_hip_yaw_link: geometry collision mesh filename=package://g1_sim/meshes/left_hip_yaw_link.STL; visual mesh filename=package://g1_sim/meshes/left_hip_yaw_link.STL
- link left_knee_link: geometry collision mesh filename=package://g1_sim/meshes/left_knee_link.STL; visual mesh filename=package://g1_sim/meshes/left_knee_link.STL
- link left_shoulder_pitch_link: geometry collision cylinder length=0.05 radius=0.03; visual mesh filename=package://g1_sim/meshes/left_shoulder_pitch_link.STL
- link left_shoulder_roll_link: geometry collision cylinder length=0.03 radius=0.03; visual mesh filename=package://g1_sim/meshes/left_shoulder_roll_link.STL
- link left_shoulder_yaw_link: geometry collision mesh filename=package://g1_sim/meshes/left_shoulder_yaw_link.STL; visual mesh filename=package://g1_sim/meshes/left_shoulder_yaw_link.STL
- link left_wrist_pitch_link: geometry collision mesh filename=package://g1_sim/meshes/left_wrist_pitch_link.STL; visual mesh filename=package://g1_sim/meshes/left_wrist_pitch_link.STL
- link left_wrist_roll_link: geometry collision mesh filename=package://g1_sim/meshes/left_wrist_roll_link.STL; visual mesh filename=package://g1_sim/meshes/left_wrist_roll_link.STL
- link left_wrist_yaw_link: geometry collision mesh filename=package://g1_sim/meshes/left_wrist_yaw_link.STL; visual mesh filename=package://g1_sim/meshes/left_wrist_yaw_link.STL
- link logo_link: geometry collision mesh filename=package://g1_sim/meshes/logo_link.STL; visual mesh filename=package://g1_sim/meshes/logo_link.STL
- link pelvis: geometry visual mesh filename=package://g1_sim/meshes/pelvis.STL
- link pelvis_contour_link: geometry collision mesh filename=package://g1_sim/meshes/pelvis_contour_link.STL; visual mesh filename=package://g1_sim/meshes/pelvis_contour_link.STL
- link right_ankle_pitch_link: geometry collision mesh filename=package://g1_sim/meshes/right_ankle_pitch_link.STL; visual mesh filename=package://g1_sim/meshes/right_ankle_pitch_link.STL
- link right_ankle_roll_link: geometry collision sphere radius=0.005; collision sphere radius=0.005
- link right_elbow_link: geometry collision mesh filename=package://g1_sim/meshes/right_elbow_link.STL; visual mesh filename=package://g1_sim/meshes/right_elbow_link.STL
- link right_hand_index_0_link: geometry collision mesh filename=package://g1_sim/meshes/right_hand_index_0_link.STL; visual mesh filename=package://g1_sim/meshes/right_hand_index_0_link.STL
- link right_hand_index_1_link: geometry collision mesh filename=package://g1_sim/meshes/right_hand_index_1_link.STL; visual mesh filename=package://g1_sim/meshes/right_hand_index_1_link.STL
- link right_hand_middle_0_link: geometry collision mesh filename=package://g1_sim/meshes/right_hand_middle_0_link.STL; visual mesh filename=package://g1_sim/meshes/right_hand_middle_0_link.STL
- link right_hand_middle_1_link: geometry collision mesh filename=package://g1_sim/meshes/right_hand_middle_1_link.STL; visual mesh filename=package://g1_sim/meshes/right_hand_middle_1_link.STL
- link right_hand_palm_link: geometry collision mesh filename=package://g1_sim/meshes/right_hand_palm_link.STL; visual mesh filename=package://g1_sim/meshes/right_hand_palm_link.STL
- link right_hand_thumb_0_link: geometry collision mesh filename=package://g1_sim/meshes/right_hand_thumb_0_link.STL; visual mesh filename=package://g1_sim/meshes/right_hand_thumb_0_link.STL
- link right_hand_thumb_1_link: geometry collision box size=0.02 0.03 0.02; visual mesh filename=package://g1_sim/meshes/right_hand_thumb_1_link.STL
- link right_hand_thumb_2_link: geometry collision mesh filename=package://g1_sim/meshes/right_hand_thumb_2_link.STL; visual mesh filename=package://g1_sim/meshes/right_hand_thumb_2_link.STL
- link right_hip_pitch_link: geometry collision mesh filename=package://g1_sim/meshes/right_hip_pitch_link.STL; visual mesh filename=package://g1_sim/meshes/right_hip_pitch_link.STL
- link right_hip_roll_link: geometry collision mesh filename=package://g1_sim/meshes/right_hip_roll_link.STL; visual mesh filename=package://g1_sim/meshes/right_hip_roll_link.STL
- link right_hip_yaw_link: geometry collision mesh filename=package://g1_sim/meshes/right_hip_yaw_link.STL; visual mesh filename=package://g1_sim/meshes/right_hip_yaw_link.STL
- link right_knee_link: geometry collision mesh filename=package://g1_sim/meshes/right_knee_link.STL; visual mesh filename=package://g1_sim/meshes/right_knee_link.STL
- link right_shoulder_pitch_link: geometry collision cylinder length=0.05 radius=0.03; visual mesh filename=package://g1_sim/meshes/right_shoulder_pitch_link.STL
- link right_shoulder_roll_link: geometry collision cylinder length=0.03 radius=0.03; visual mesh filename=package://g1_sim/meshes/right_shoulder_roll_link.STL
- link right_shoulder_yaw_link: geometry collision mesh filename=package://g1_sim/meshes/right_shoulder_yaw_link.STL; visual mesh filename=package://g1_sim/meshes/right_shoulder_yaw_link.STL
- link right_wrist_pitch_link: geometry collision mesh filename=package://g1_sim/meshes/right_wrist_pitch_link.STL; visual mesh filename=package://g1_sim/meshes/right_wrist_pitch_link.STL
- link right_wrist_roll_link: geometry collision mesh filename=package://g1_sim/meshes/right_wrist_roll_link.STL; visual mesh filename=package://g1_sim/meshes/right_wrist_roll_link.STL
- link right_wrist_yaw_link: geometry collision mesh filename=package://g1_sim/meshes/right_wrist_yaw_link.STL; visual mesh filename=package://g1_sim/meshes/right_wrist_yaw_link.STL
- link torso_link: geometry collision mesh filename=package://g1_sim/meshes/torso_link.STL; visual mesh filename=package://g1_sim/meshes/torso_link.STL
- link waist_roll_link: geometry visual mesh filename=package://g1_sim/meshes/waist_roll_link.STL
- link waist_support_link: geometry collision mesh filename=package://g1_sim/meshes/waist_support_link.STL; visual mesh filename=package://g1_sim/meshes/waist_support_link.STL
- link waist_yaw_link: geometry visual mesh filename=package://g1_sim/meshes/waist_yaw_link.STL

Commit message: g1 2d激光建图调试

File: unitree_g1_ros2_function_pkg/src/g1_sim/urdf/g1_29dof_with_hand.urdf (robot description, URDF)
Before this commit: robot g1_29dof_with_hand, 54 links, 53 joints
Links:
- removed link pelvis
- added link base, mass 3.813; visual mesh filename=package://g1_sim/meshes/pelvis.STL
Joints:
- joint imu_in_pelvis_joint: parent pelvis -> base
- joint left_hip_pitch_joint: parent pelvis -> base
- joint pelvis_contour_joint: parent pelvis -> base
- joint right_hip_pitch_joint: parent pelvis -> base
- joint waist_yaw_joint: parent pelvis -> base

Commit message: g1实机调试

File: unitree_g1_ros2_function_pkg/src/g1_sim/urdf/g1_29dof_with_hand.urdf (robot description, URDF)
Before this commit: robot g1_29dof_with_hand, 54 links, 53 joints
Links:
- removed link d435_link
- added link camera_link
Joints:
- joint d435_joint: child d435_link -> camera_link
